Commit message: Added claw for future animations and changed color

File: urdf/pa10.urdf.xacro (robot description, xacro)
@@ -44,5 +44,5 @@
       </geometry>
 	<material name="">
-        <color rgba="0.33 0.96 0.53 1.0"/>
+        <color rgba="0.7 0.0 0.0 1.0"/>
       </material>
     </visual>
@@ -94,5 +94,5 @@
       </geometry>
 	<material name="">
-        <color rgba="0.33 0.96 0.53 1.0"/>
+        <color rgba="0.7 0.0 0.0 1.0"/>
       </material>
     </visual>
@@ -144,5 +144,5 @@
       </geometry>
 	<material name="">
-        <color rgba="0.33 0.96 0.53 1.0"/>
+        <color rgba="0.7 0.0 0.0 1.0"/>
       </material>
     </visual>
@@ -187,5 +187,82 @@
     </inertial>
   </link>
-  <link name = "ee_link"/>
+  <link name="ee_link">
+    <inertial>
+      <mass value="0.1"/>
+      <origin xyz="0 0 0" rpy="0 0 0"/>
+      <inertia ixx="0.001" iyy="0.001" izz="0.001" ixy="0.0" ixz="0.0" iyz="0.0"/>
+    </inertial>
+  </link>
+  <link name="link_gripper_base">
+    <visual>
+      <origin rpy="0 0 0" xyz="0 0 -0.045"/>
+      <geometry>
+        <mesh filename="file://$(find manipulatorws)/meshes/gripper_stl/pa10_gripper_base.stl"/>
+      </geometry>
+      <material name="">
+        <color rgba="0.8 0.0 0.0 1.0"/> <!-- red for visibility -->
+      </material>
+    </visual>
+    <collision>
+      <origin rpy="0 0 0" xyz="0 0 -0.045"/>
+      <geometry>
+        <mesh filename="file://$(find manipulatorws)/meshes/gripper_stl/pa10_gripper_base.stl"/>
+      </geometry>
+    </collision>
+    <inertial>
+      <origin xyz="0 0 0" rpy="0 0 0"/>
+      <mass value="0.2"/>
+      <inertia
+        ixx="0.001" ixy="0.0" ixz="0.0"
+        iyy="0.001" iyz="0.0"
+        izz="0.001"/>
+    </inertial>
+  </link>
+        <link name="link_finger_1">
+            <visual>
+                <origin rpy="-3.14159 -1.57079 0" xyz="-0.0225 0.075 -0.01"/>
+                <geometry>
+                    <mesh filename="file://$(find manipulatorws)/meshes/gripper_stl/finger.stl" scale="0.001 0.001 0.001"/>
+                </geometry>
+                <material name="">
+                  <color rgba="0.9 0.75 0.3 1.0"/>
+                </material>
+            </visual>
+            <collision>
+                <origin rpy="-3.14159 -1.57079 0" xyz="-0.0225 0.075 -0.01"/>
+                <geometry>
+                    <mesh filename="file://$(find manipulatorws)/meshes/gripper_stl/finger.stl" scale="0.001 0.001 0.001"/>
+                </geometry>
+            </collision>
+            <!--inertial-->
+                <!--mass value="${mass_gripper}"/-->
+                <!-- <inertia ixx="0.01" ixy="0.0" ixz="0.0" iyy="0.01" iyz="0.0" izz="0.01"/> -->
+                <!-- <xacro:inertia_box height="${inertia_height_gripper}" mass="${mass_gripper}"/> -->
+                <!--inertia ixx="0.1" ixy="0.0" ixz="0.0" iyy="0.1" iyz="0.0" izz="0.1"/-->
+            <!--inertial-->
+        </link>
+        <link name="link_finger_2">
+            <visual>
+                <origin rpy="0 1.57079 0" xyz="-0.0225 -0.075 0.07"/>
+                <geometry>
+                    <mesh filename="file://$(find manipulatorws)/meshes/gripper_stl/finger_left.stl" scale="0.001 0.001 0.001"/>
+                </geometry>
+                <material name="">
+                  <color rgba="0.9 0.75 0.3 1.0"/>
+                </material>
+            </visual>
+            <collision>
+                <origin rpy="0 1.57079 0" xyz="-0.0225 -0.075 0.07"/>
+                <geometry>
+                    <mesh filename="file://$(find manipulatorws)/meshes/gripper_stl/finger_left.stl" scale="0.001 0.001 0.001"/>
+                </geometry>
+            </collision>
+            <!--inertial-->
+                <!--mass value="${mass_gripper}"/-->
+                <!-- <inertia ixx="0.01" ixy="0.0" ixz="0.0" iyy="0.01" iyz="0.0" izz="0.01"/> -->
+                <!-- <xacro:inertia_box height="${inertia_height_gripper}" mass="${mass_gripper}"/> -->
+                <!--inertia ixx="0.1" ixy="0.0" ixz="0.0" iyy="0.1" iyz="0.0" izz="0.1"/-->
+            <!--/inertial-->
+        </link>
 <joint name="S1" type="revolute">
     <origin rpy="0 0 0" xyz="0 0 0.2"/>
@@ -237,3 +314,22 @@
     <limit effort="0" lower="-2.878" upper="2.878" velocity="1.0"/>
   </joint>
+  <joint name="gripper_joint" type="fixed">
+    <origin rpy="0 0 0" xyz="0 0 0.045"/>
+    <parent link="ee_link"/>
+    <child link="link_gripper_base"/>
+  </joint>
+<joint name="finger_1_joint" type="prismatic">
+  <parent link="link_gripper_base"/>
+  <child link="link_finger_1"/>
+  <origin rpy="-1.57079 0 0" xyz="0 ${-0.03-0.01} 0.11"/>
+  <axis xyz="0 0 1"/> <!-- Moves along Y-axis (adjust if necessary) -->
+  <limit lower="0.0" upper="0.02" effort="10.0" velocity="0.02"/>
+</joint>
+<joint name="finger_2_joint" type="prismatic">
+  <parent link="link_gripper_base"/>
+  <child link="link_finger_2"/>
+  <origin rpy="1.57079 0 0" xyz="0 ${0.03+0.01} 0.11"/>
+  <axis xyz="0 0 1"/> <!-- Opposite direction to finger_1 -->
+  <limit lower="0.0" upper="0.02" effort="10.0" velocity="0.02"/>
+</joint>
 </robot>

Commit message: Working on gazebo simulations

File: urdf/pa10.urdf.xacro (robot description, xacro)
@@ -235,10 +235,12 @@
                 </geometry>
             </collision>
-            <!--inertial-->
-                <!--mass value="${mass_gripper}"/-->
-                <!-- <inertia ixx="0.01" ixy="0.0" ixz="0.0" iyy="0.01" iyz="0.0" izz="0.01"/> -->
-                <!-- <xacro:inertia_box height="${inertia_height_gripper}" mass="${mass_gripper}"/> -->
-                <!--inertia ixx="0.1" ixy="0.0" ixz="0.0" iyy="0.1" iyz="0.0" izz="0.1"/-->
-            <!--inertial-->
+          <inertial>
+            <origin xyz="0 0 0" rpy="0 0 0"/>
+            <mass value="0.01"/>
+            <inertia
+              ixx="0.00001" ixy="0.0" ixz="0.0"
+              iyy="0.00001" iyz="0.0"
+              izz="0.00001"/>
+          </inertial>
         </link>
         <link name="link_finger_2">
@@ -258,10 +260,12 @@
                 </geometry>
             </collision>
-            <!--inertial-->
-                <!--mass value="${mass_gripper}"/-->
-                <!-- <inertia ixx="0.01" ixy="0.0" ixz="0.0" iyy="0.01" iyz="0.0" izz="0.01"/> -->
-                <!-- <xacro:inertia_box height="${inertia_height_gripper}" mass="${mass_gripper}"/> -->
-                <!--inertia ixx="0.1" ixy="0.0" ixz="0.0" iyy="0.1" iyz="0.0" izz="0.1"/-->
-            <!--/inertial-->
+              <inertial>
+                <origin xyz="0 0 0" rpy="0 0 0"/>
+                <mass value="0.01"/>
+                <inertia
+                  ixx="0.00001" ixy="0.0" ixz="0.0"
+                  iyy="0.00001" iyz="0.0"
+                  izz="0.00001"/>
+              </inertial>
         </link>
 <joint name="S1" type="revolute">

Commit message: Finally got it working with gazebo, extensive notes must be taken

File: urdf/pa10.urdf.xacro (robot description, xacro)
@@ -1,5 +1,4 @@
 <?xml version="1.0" ?>
 <robot name="pa10" xmlns:xacro="http://www.ros.org/wiki/xacro">
-	<!-- Used for fixing robot to Gazebo 'base_link' -->
   <link name="world"/>
   <joint name="fixed" type="fixed">
@@ -269,71 +268,71 @@
               </inertial>
         </link>
-<joint name="S1" type="revolute">
-    <origin rpy="0 0 0" xyz="0 0 0.2"/>
-    <parent link="base_link"/>
-    <child link="link_1"/>
-    <axis xyz="0 0 1"/>
-    <limit effort="0" lower="-3.089" upper="3.089" velocity="1.0"/>
+  <joint name="S1" type="revolute">
+      <origin rpy="0 0 0" xyz="0 0 0.2"/>
+      <parent link="base_link"/>
+      <child link="link_1"/>
+      <axis xyz="0 0 1"/>
+      <limit effort="100" lower="-3.089" upper="3.089" velocity="1.0"/>
+    </joint>
+  <joint name="S2" type="revolute">
+      <origin rpy="0 0 0" xyz="0 0 0.117"/>
+      <parent link="link_1"/>
+      <child link="link_2"/>
+      <axis xyz="0 1 0"/>
+      <limit effort="100" lower="-1.64" upper="1.64" velocity="1.0"/>
+    </joint>
+  <joint name="S3" type="revolute">
+      <origin rpy="0 0 0" xyz="0 0 0.317"/>
+      <parent link="link_2"/>
+      <child link="link_3"/>
+      <axis xyz="0 0 1"/>
+      <limit effort="100" lower="-3.036" upper="3.036" velocity="1.0"/>
+    </joint>
+  <joint name="E1" type="revolute">
+      <origin rpy="0 0 0" xyz="0 0 0.133"/>
+      <parent link="link_3"/>
+      <child link="link_4"/>
+      <axis xyz="0 1 0"/>
+      <limit effort="100" lower="-2.39" upper="2.39" velocity="1.0"/>
+    </joint>
+  <joint name="E2" type="revolute">
+      <origin rpy="0 0 0" xyz="0 0 0.285"/>
+      <parent link="link_4"/>
+      <child link="link_5"/>
+      <axis xyz="0 0 1"/>
+      <limit effort="100" lower="-4.45" upper="4.45" velocity="1.0"/>
+    </joint>
+  <joint name="W1" type="revolute">
+      <origin rpy="0 0 0" xyz="0 0 0.195"/>
+      <parent link="link_5"/>
+      <child link="link_6"/>
+      <axis xyz="0 1 0"/>
+      <limit effort="100" lower="-2.878" upper="2.878" velocity="1.0"/>
+    </joint>
+    <joint name = "W2" type="revolute">
+      <origin rpy="0 0 0" xyz="0 0 0"/>
+      <parent link="link_6"/>
+      <child link="ee_link"/>
+      <axis xyz="0 0 1"/>
+      <limit effort="100" lower="-2.878" upper="2.878" velocity="1.0"/>
+    </joint>
+    <joint name="gripper_joint" type="fixed">
+      <origin rpy="0 0 0" xyz="0 0 0.045"/>
+      <parent link="ee_link"/>
+      <child link="link_gripper_base"/>
+    </joint>
+  <joint name="finger_1_joint" type="prismatic">
+    <parent link="link_gripper_base"/>
+    <child link="link_finger_1"/>
+    <origin rpy="-1.57079 0 0" xyz="0 -0.04 0.11"/>
+    <axis xyz="0 0 1"/> <!-- Moves along Y-axis (adjust if necessary) -->
+    <limit lower="0.0" upper="0.02" effort="10.0" velocity="0.02"/>
   </joint>
-<joint name="S2" type="revolute">
-    <origin rpy="0 0 0" xyz="0 0 0.117"/>
-    <parent link="link_1"/>
-    <child link="link_2"/>
-    <axis xyz="0 1 0"/>
-    <limit effort="0" lower="-1.64" upper="1.64" velocity="1.0"/>
+  <joint name="finger_2_joint" type="prismatic">
+    <parent link="link_gripper_base"/>
+    <child link="link_finger_2"/>
+    <origin rpy="1.57079 0 0" xyz="0 0.04 0.11"/>
+    <axis xyz="0 0 1"/> <!-- Opposite direction to finger_1 -->
+    <limit lower="0.0" upper="0.02" effort="10.0" velocity="0.02"/>
   </joint>
-<joint name="S3" type="revolute">
-    <origin rpy="0 0 0" xyz="0 0 0.317"/>
-    <parent link="link_2"/>
-    <child link="link_3"/>
-    <axis xyz="0 0 1"/>
-    <limit effort="0" lower="-3.036" upper="3.036" velocity="1.0"/>
-  </joint>
-<joint name="E1" type="revolute">
-    <origin rpy="0 0 0" xyz="0 0 0.133"/>
-    <parent link="link_3"/>
-    <child link="link_4"/>
-    <axis xyz="0 1 0"/>
-    <limit effort="0" lower="-2.39" upper="2.39" velocity="1.0"/>
-  </joint>
-<joint name="E2" type="revolute">
-    <origin rpy="0 0 0" xyz="0 0 0.285"/>
-    <parent link="link_4"/>
-    <child link="link_5"/>
-    <axis xyz="0 0 1"/>
-    <limit effort="0" lower="-4.45" upper="4.45" velocity="1.0"/>
-  </joint>
-<joint name="W1" type="revolute">
-    <origin rpy="0 0 0" xyz="0 0 0.195"/>
-    <parent link="link_5"/>
-    <child link="link_6"/>
-    <axis xyz="0 1 0"/>
-    <limit effort="0" lower="-2.878" upper="2.878" velocity="1.0"/>
-  </joint>
-  <joint name = "W2" type="revolute">
-    <origin rpy="0 0 0" xyz="0 0 0"/>
-    <parent link="link_6"/>
-    <child link="ee_link"/>
-    <axis xyz="0 0 1"/>
-    <limit effort="0" lower="-2.878" upper="2.878" velocity="1.0"/>
-  </joint>
-  <joint name="gripper_joint" type="fixed">
-    <origin rpy="0 0 0" xyz="0 0 0.045"/>
-    <parent link="ee_link"/>
-    <child link="link_gripper_base"/>
-  </joint>
-<joint name="finger_1_joint" type="prismatic">
-  <parent link="link_gripper_base"/>
-  <child link="link_finger_1"/>
-  <origin rpy="-1.57079 0 0" xyz="0 ${-0.03-0.01} 0.11"/>
-  <axis xyz="0 0 1"/> <!-- Moves along Y-axis (adjust if necessary) -->
-  <limit lower="0.0" upper="0.02" effort="10.0" velocity="0.02"/>
-</joint>
-<joint name="finger_2_joint" type="prismatic">
-  <parent link="link_gripper_base"/>
-  <child link="link_finger_2"/>
-  <origin rpy="1.57079 0 0" xyz="0 ${0.03+0.01} 0.11"/>
-  <axis xyz="0 0 1"/> <!-- Opposite direction to finger_1 -->
-  <limit lower="0.0" upper="0.02" effort="10.0" velocity="0.02"/>
-</joint>
 </robot>

Commit message: node to node communication now works

File: urdf/pa10.urdf.xacro (robot description, xacro)
@@ -321,4 +321,5 @@
       <parent link="ee_link"/>
       <child link="link_gripper_base"/>
+      <limit effort="100" lower="-2.878" upper="2.878" velocity="1.0"/>
     </joint>
   <joint name="finger_1_joint" type="prismatic">

Commit message: adding gif

File: urdf/pa10.urdf.xacro (robot description, xacro)
@@ -328,5 +328,5 @@
     <origin rpy="-1.57079 0 0" xyz="0 -0.04 0.11"/>
     <axis xyz="0 0 1"/> <!-- Moves along Y-axis (adjust if necessary) -->
-    <limit lower="0.0" upper="0.02" effort="10.0" velocity="0.02"/>
+    <limit lower="100.0" upper="0.02" effort="10.0" velocity="0.02"/>
   </joint>
   <joint name="finger_2_joint" type="prismatic">
@@ -335,5 +335,5 @@
     <origin rpy="1.57079 0 0" xyz="0 0.04 0.11"/>
     <axis xyz="0 0 1"/> <!-- Opposite direction to finger_1 -->
-    <limit lower="0.0" upper="0.02" effort="10.0" velocity="0.02"/>
+    <limit lower="100.0" upper="0.02" effort="10.0" velocity="0.02"/>
   </joint>
 </robot>
