Commit message: dual arm urdf file done

File: urdf/pa10.urdf.xacro (robot description, xacro)
@@ -1,339 +1,339 @@
 <?xml version="1.0" ?>
 <robot name="pa10" xmlns:xacro="http://www.ros.org/wiki/xacro">
-  <link name="world"/>
-  <joint name="fixed" type="fixed">
-    <parent link="world"/>
-    <child link="base_link"/>
-  </joint>
-	<!-- Import all Gazebo-customization elements, including Gazebo colors -->
-  <!--xacro:include filename="$(find pa10_description)/urdf/pa10.gazebo" -->
-  <!-- Import Rviz colors -->
-  <!--xacro:include filename="file://$(find manipulatorws)/urdf/materials.xacro" /-->
-  <link name="base_link">
-    <visual>
-      <origin rpy="0 0 3.14" xyz="0 0 0"/>
-      <geometry>
-        <mesh filename="file://$(find manipulatorws)/meshes/pa10_stl/S1.stl"/>
-<!-- podemos usar tambien en vez de mesh que requiere un archivo, cilindros cajas o esferas!!! -->
-      </geometry>
-      <material name="">
-        <color rgba="0.34 0.35 0.36 1.0"/>
-      </material>
-    </visual>
-    <collision>
-      <origin rpy="0 0 3.14" xyz="0 0 0"/>
-      <geometry>
-        <mesh filename="file://$(find manipulatorws)/meshes/pa10_stl_collision/S1_collision.stl"/>
-      </geometry>
-    </collision>
-    <inertial>
-      <origin xyz="0 0 1" rpy="0 0 0"/>
-      <mass value="1"/>
-      <inertia
-	  ixx="1" ixy="0.0" ixz="0.0"
-	  iyy="1" iyz="0.0"
-	  izz="1"/>
-    </inertial>
-  </link>
-<link name="link_1">
-    <visual>
-      <origin rpy="0 0 0" xyz="0 0 0.117"/>
-      <geometry>
-        <mesh filename="file://$(find manipulatorws)/meshes/pa10_stl/S2.stl"/>
-      </geometry>
-	<material name="">
-        <color rgba="0.7 0.0 0.0 1.0"/>
-      </material>
-    </visual>
-    <collision>
-      <origin rpy="0 0 0" xyz="0 0 0.117"/>
-      <geometry>
-        <mesh filename="file://$(find manipulatorws)/meshes/pa10_stl_collision/S2_collision.stl"/>
-      </geometry>
-    </collision>
-    <inertial>
-      <origin xyz="0 0 1" rpy="0 0 0"/>
-      <mass value="1"/>
-      <inertia
-	  ixx="1" ixy="0.0" ixz="0.0"
-	  iyy="1" iyz="0.0"
-	  izz="1"/>
-    </inertial>
-  </link>
-<link name="link_2">
-    <visual>
-      <origin rpy="0 0 0" xyz="0 0 0"/>
-      <geometry>
-        <mesh filename="file://$(find manipulatorws)/meshes/pa10_stl/S3.stl"/>
-      </geometry>
-      <material name="">
-        <color rgba="0.34 0.35 0.36 1.0"/>
-      </material>
-    </visual>
-    <collision>
-      <origin rpy="0 0 0" xyz="0 0 0"/>
-      <geometry>
-        <mesh filename="file://$(find manipulatorws)/meshes/pa10_stl_collision/S3_collision.stl"/>
-      </geometry>
-    </collision>
-    <inertial>
-      <origin xyz="0 0 1" rpy="0 0 0"/>
-      <mass value="1"/>
-      <inertia
-	  ixx="1" ixy="0.0" ixz="0.0"
-	  iyy="1" iyz="0.0"
-	  izz="1"/>
-    </inertial>
-  </link>
-<link name="link_3">
-    <visual>
-      <origin rpy="0 0 0" xyz="0 0 0.133"/>
-      <geometry>
-        <mesh filename="file://$(find manipulatorws)/meshes/pa10_stl/E1.stl"/>
-      </geometry>
-	<material name="">
-        <color rgba="0.7 0.0 0.0 1.0"/>
-      </material>
-    </visual>
-    <collision>
-      <origin rpy="0 0 0" xyz="0 0 0.133"/>
-      <geometry>
-        <mesh filename="file://$(find manipulatorws)/meshes/pa10_stl_collision/E1_collision.stl"/>
-      </geometry>
-    </collision>
-    <inertial>
-      <origin xyz="0 0 1" rpy="0 0 0"/>
-      <mass value="1"/>
-      <inertia
-	  ixx="1" ixy="0.0" ixz="0.0"
-	  iyy="1" iyz="0.0"
-	  izz="1"/>
-    </inertial>
-  </link>
-<link name="link_4">
-    <visual>
-      <origin rpy="0 0 0" xyz="0 0.003 0"/>
-      <geometry>
-        <mesh filename="file://$(find manipulatorws)/meshes/pa10_stl/E2.stl"/>
-      </geometry>
-	<material name="">
-        <color rgba="0.34 0.35 0.36 1.0"/>
-      </material>
-    </visual>
-    <collision>
-      <origin rpy="0 0 0" xyz="0 0.003 0"/>
-      <geometry>
-        <mesh filename="file://$(find manipulatorws)/meshes/pa10_stl_collision/E2_collision.stl"/>
-      </geometry>
-    </collision>
-    <inertial>
-      <origin xyz="0 0 1" rpy="0 0 0"/>
-      <mass value="1"/>
-      <inertia
-	  ixx="1" ixy="0.0" ixz="0.0"
-	  iyy="1" iyz="0.0"
-	  izz="1"/>
-    </inertial>
-  </link>
-<link name="link_5">
-    <visual>
-      <origin rpy="0 0 0" xyz="0 0 0.195"/>
-      <geometry>
-        <mesh filename="file://$(find manipulatorws)/meshes/pa10_stl/W1.stl"/>
-      </geometry>
-	<material name="">
-        <color rgba="0.7 0.0 0.0 1.0"/>
-      </material>
-    </visual>
-    <collision>
-      <origin rpy="0 0 0" xyz="0 0 0.195"/>
-      <geometry>
-        <mesh filename="file://$(find manipulatorws)/meshes/pa10_stl_collision/W1_collision.stl"/>
-      </geometry>
-    </collision>
-    <inertial>
-      <origin xyz="0 0 1" rpy="0 0 0"/>
-      <mass value="1"/>
-      <inertia
-	  ixx="1" ixy="0.0" ixz="0.0"
-	  iyy="1" iyz="0.0"
-	  izz="1"/>
-    </inertial>
-  </link>
-<link name="link_6">
-    <visual>
-      <origin rpy="0 0 0" xyz="0 0 0"/>
-      <geometry>
-        <mesh filename="file://$(find manipulatorws)/meshes/pa10_stl/W2.stl"/>
-      </geometry>
-	<material name="">
-        <color rgba="0.34 0.35 0.36 1.0"/>
-      </material>
-    </visual>
-    <collision>
-      <origin rpy="0 0 0" xyz="0 0 0"/>
-      <geometry>
-        <mesh filename="file://$(find manipulatorws)/meshes/pa10_stl_collision/W2_collision.stl"/>
-      </geometry>
-    </collision>
-    <inertial>
-      <origin xyz="0 0 1" rpy="0 0 0"/>
-      <mass value="1"/>
-      <inertia
-	  ixx="1" ixy="0.0" ixz="0.0"
-	  iyy="1" iyz="0.0"
-	  izz="1"/>
-    </inertial>
-  </link>
-  <link name="ee_link">
-    <inertial>
-      <mass value="0.1"/>
-      <origin xyz="0 0 0" rpy="0 0 0"/>
-      <inertia ixx="0.001" iyy="0.001" izz="0.001" ixy="0.0" ixz="0.0" iyz="0.0"/>
-    </inertial>
-  </link>
-  <link name="link_gripper_base">
-    <visual>
-      <origin rpy="0 0 0" xyz="0 0 -0.045"/>
-      <geometry>
-        <mesh filename="file://$(find manipulatorws)/meshes/gripper_stl/pa10_gripper_base.stl"/>
-      </geometry>
-      <material name="">
-        <color rgba="0.8 0.0 0.0 1.0"/> <!-- red for visibility -->
-      </material>
-    </visual>
-    <collision>
-      <origin rpy="0 0 0" xyz="0 0 -0.045"/>
-      <geometry>
-        <mesh filename="file://$(find manipulatorws)/meshes/gripper_stl/pa10_gripper_base.stl"/>
-      </geometry>
-    </collision>
-    <inertial>
-      <origin xyz="0 0 0" rpy="0 0 0"/>
-      <mass value="0.2"/>
-      <inertia
-        ixx="0.001" ixy="0.0" ixz="0.0"
-        iyy="0.001" iyz="0.0"
-        izz="0.001"/>
-    </inertial>
-  </link>
-        <link name="link_finger_1">
-            <visual>
-                <origin rpy="-3.14159 -1.57079 0" xyz="-0.0225 0.075 -0.01"/>
-                <geometry>
-                    <mesh filename="file://$(find manipulatorws)/meshes/gripper_stl/finger.stl" scale="0.001 0.001 0.001"/>
-                </geometry>
-                <material name="">
-                  <color rgba="0.9 0.75 0.3 1.0"/>
-                </material>
-            </visual>
-            <collision>
-                <origin rpy="-3.14159 -1.57079 0" xyz="-0.0225 0.075 -0.01"/>
-                <geometry>
-                    <mesh filename="file://$(find manipulatorws)/meshes/gripper_stl/finger.stl" scale="0.001 0.001 0.001"/>
-                </geometry>
-            </collision>
-          <inertial>
-            <origin xyz="0 0 0" rpy="0 0 0"/>
-            <mass value="0.01"/>
-            <inertia
-              ixx="0.00001" ixy="0.0" ixz="0.0"
-              iyy="0.00001" iyz="0.0"
-              izz="0.00001"/>
-          </inertial>
-        </link>
-        <link name="link_finger_2">
-            <visual>
-                <origin rpy="0 1.57079 0" xyz="-0.0225 -0.075 0.07"/>
-                <geometry>
-                    <mesh filename="file://$(find manipulatorws)/meshes/gripper_stl/finger_left.stl" scale="0.001 0.001 0.001"/>
-                </geometry>
-                <material name="">
-                  <color rgba="0.9 0.75 0.3 1.0"/>
-                </material>
-            </visual>
-            <collision>
-                <origin rpy="0 1.57079 0" xyz="-0.0225 -0.075 0.07"/>
-                <geometry>
-                    <mesh filename="file://$(find manipulatorws)/meshes/gripper_stl/finger_left.stl" scale="0.001 0.001 0.001"/>
-                </geometry>
-            </collision>
-              <inertial>
-                <origin xyz="0 0 0" rpy="0 0 0"/>
-                <mass value="0.01"/>
-                <inertia
-                  ixx="0.00001" ixy="0.0" ixz="0.0"
-                  iyy="0.00001" iyz="0.0"
-                  izz="0.00001"/>
-              </inertial>
-        </link>
-  <joint name="S1" type="revolute">
-      <origin rpy="0 0 0" xyz="0 0 0.2"/>
-      <parent link="base_link"/>
-      <child link="link_1"/>
-      <axis xyz="0 0 1"/>
-      <limit effort="100" lower="-3.089" upper="3.089" velocity="1.0"/>
+  <xacro:macro name="pa10_arm" params="prefix parent xyz rpy">
+    <joint name="${prefix}base_fixed_joint" type="fixed">
+      <parent link="${parent}"/>
+      <child link="${prefix}base_link"/>
+      <origin xyz="${xyz}" rpy="${rpy}"/>
     </joint>
-  <joint name="S2" type="revolute">
-      <origin rpy="0 0 0" xyz="0 0 0.117"/>
-      <parent link="link_1"/>
-      <child link="link_2"/>
-      <axis xyz="0 1 0"/>
-      <limit effort="100" lower="-1.64" upper="1.64" velocity="1.0"/>
-    </joint>
-  <joint name="S3" type="revolute">
-      <origin rpy="0 0 0" xyz="0 0 0.317"/>
-      <parent link="link_2"/>
-      <child link="link_3"/>
-      <axis xyz="0 0 1"/>
-      <limit effort="100" lower="-3.036" upper="3.036" velocity="1.0"/>
-    </joint>
-  <joint name="E1" type="revolute">
-      <origin rpy="0 0 0" xyz="0 0 0.133"/>
-      <parent link="link_3"/>
-      <child link="link_4"/>
-      <axis xyz="0 1 0"/>
-      <limit effort="100" lower="-2.39" upper="2.39" velocity="1.0"/>
-    </joint>
-  <joint name="E2" type="revolute">
-      <origin rpy="0 0 0" xyz="0 0 0.285"/>
-      <parent link="link_4"/>
-      <child link="link_5"/>
-      <axis xyz="0 0 1"/>
-      <limit effort="100" lower="-4.45" upper="4.45" velocity="1.0"/>
-    </joint>
-  <joint name="W1" type="revolute">
-      <origin rpy="0 0 0" xyz="0 0 0.195"/>
-      <parent link="link_5"/>
-      <child link="link_6"/>
-      <axis xyz="0 1 0"/>
-      <limit effort="100" lower="-2.878" upper="2.878" velocity="1.0"/>
-    </joint>
-    <joint name = "W2" type="revolute">
-      <origin rpy="0 0 0" xyz="0 0 0"/>
-      <parent link="link_6"/>
-      <child link="ee_link"/>
-      <axis xyz="0 0 1"/>
-      <limit effort="100" lower="-2.878" upper="2.878" velocity="1.0"/>
-    </joint>
-    <joint name="gripper_joint" type="fixed">
-      <origin rpy="0 0 0" xyz="0 0 0.045"/>
-      <parent link="ee_link"/>
-      <child link="link_gripper_base"/>
-      <limit effort="100" lower="-2.878" upper="2.878" velocity="1.0"/>
-    </joint>
-  <joint name="finger_1_joint" type="prismatic">
-    <parent link="link_gripper_base"/>
-    <child link="link_finger_1"/>
-    <origin rpy="-1.57079 0 0" xyz="0 -0.04 0.11"/>
-    <axis xyz="0 0 1"/> <!-- Moves along Y-axis (adjust if necessary) -->
-    <limit lower="100.0" upper="0.02" effort="10.0" velocity="0.02"/>
-  </joint>
-  <joint name="finger_2_joint" type="prismatic">
-    <parent link="link_gripper_base"/>
-    <child link="link_finger_2"/>
-    <origin rpy="1.57079 0 0" xyz="0 0.04 0.11"/>
-    <axis xyz="0 0 1"/> <!-- Opposite direction to finger_1 -->
-    <limit lower="100.0" upper="0.02" effort="10.0" velocity="0.02"/>
-  </joint>
+    <!-- Import all Gazebo-customization elements, including Gazebo colors -->
+    <!--xacro:include filename="$(find pa10_description)/urdf/pa10.gazebo" -->
+    <!-- Import Rviz colors -->
+    <!--xacro:include filename="file://$(find manipulatorws)/urdf/materials.xacro" /-->
+    <link name="${prefix}base_link">
+      <visual>
+        <origin rpy="0 0 3.14" xyz="0 0 0"/>
+        <geometry>
+          <mesh filename="file://$(find manipulatorws)/meshes/pa10_stl/S1.stl"/>
+        </geometry>
+        <material name="">
+          <color rgba="0.34 0.35 0.36 1.0"/>
+        </material>
+      </visual>
+      <collision>
+        <origin rpy="0 0 3.14" xyz="0 0 0"/>
+        <geometry>
+          <mesh filename="file://$(find manipulatorws)/meshes/pa10_stl_collision/S1_collision.stl"/>
+        </geometry>
+      </collision>
+      <inertial>
+        <origin xyz="0 0 1" rpy="0 0 0"/>
+        <mass value="1"/>
+        <inertia
+      ixx="1" ixy="0.0" ixz="0.0"
+      iyy="1" iyz="0.0"
+      izz="1"/>
+      </inertial>
+    </link>
+  <link name="${prefix}link_1">
+      <visual>
+        <origin rpy="0 0 0" xyz="0 0 0.117"/>
+        <geometry>
+          <mesh filename="file://$(find manipulatorws)/meshes/pa10_stl/S2.stl"/>
+        </geometry>
+    <material name="">
+          <color rgba="0.7 0.0 0.0 1.0"/>
+        </material>
+      </visual>
+      <collision>
+        <origin rpy="0 0 0" xyz="0 0 0.117"/>
+        <geometry>
+          <mesh filename="file://$(find manipulatorws)/meshes/pa10_stl_collision/S2_collision.stl"/>
+        </geometry>
+      </collision>
+      <inertial>
+        <origin xyz="0 0 1" rpy="0 0 0"/>
+        <mass value="1"/>
+        <inertia
+      ixx="1" ixy="0.0" ixz="0.0"
+      iyy="1" iyz="0.0"
+      izz="1"/>
+      </inertial>
+    </link>
+  <link name="${prefix}link_2">
+      <visual>
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
File: urdf/pa10_gazebo.urdf.xacro (robot description, xacro)
@@ -3,9 +3,10 @@
   <!-- Arguments -->
   <xacro:arg name="robot_name" default="pa10"/>
-  <xacro:arg name="add_world" default="true"/>
   <xacro:arg name="use_gazebo" default="true"/>
-  <!-- Include visuals, links, and joints -->
+  <!-- Include arm macro definition -->
   <xacro:include filename="$(find manipulatorws)/urdf/pa10.urdf.xacro"/>
-  <!-- Optional gripper is already inside pa10.urdf.xacro -->
+  <link name="world"/>
+  <!-- Instantiate the robot arm -->
+  <xacro:pa10_arm prefix="" parent="world" xyz="0 0 0" rpy="0 0 0"/>
   <!-- Load ROS2 Control plugin for Gazebo -->
   <xacro:include filename="$(find manipulatorws)/urdf/controls/gazebo_sim_ros2_control.urdf.xacro"/>

Commit message: updated gazebo world and link colors

File: urdf/pa10.urdf.xacro (robot description, xacro)
@@ -18,5 +18,5 @@
         </geometry>
         <material name="">
-          <color rgba="0.34 0.35 0.36 1.0"/>
+          <color rgba="0.1 0.9 1.0 0.4"/> <!-- Bright cyan glow, semi-transparent -->
         </material>
       </visual>
@@ -42,34 +42,34 @@
           <mesh filename="file://$(find manipulatorws)/meshes/pa10_stl/S2.stl"/>
         </geometry>
-    <material name="">
-          <color rgba="0.7 0.0 0.0 1.0"/>
+      <material name="">
+        <color rgba="0.0 1.0 1.0 0.4"/> <!-- RGB = Cyan, A = 30% visible -->
+      </material>
+      </visual>
+      <collision>
+        <origin rpy="0 0 0" xyz="0 0 0.117"/>
+        <geometry>
+          <mesh filename="file://$(find manipulatorws)/meshes/pa10_stl_collision/S2_collision.stl"/>
+        </geometry>
+      </collision>
+      <inertial>
+        <origin xyz="0 0 1" rpy="0 0 0"/>
+        <mass value="1"/>
+        <inertia
+      ixx="1" ixy="0.0" ixz="0.0"
+      iyy="1" iyz="0.0"
+      izz="1"/>
+      </inertial>
+    </link>
+  <link name="${prefix}link_2">
+      <visual>
+        <origin rpy="0 0 0" xyz="0 0 0"/>
+        <geometry>
+          <mesh filename="file://$(find manipulatorws)/meshes/pa10_stl/S3.stl"/>
+        </geometry>
+        <material name="">
+          <color rgba="0.0 1.0 1.0 0.4"/> <!-- RGB = Cyan, A = 30% visible -->
         </material>
       </visual>
       <collision>
-        <origin rpy="0 0 0" xyz="0 0 0.117"/>
-        <geometry>
-          <mesh filename="file://$(find manipulatorws)/meshes/pa10_stl_collision/S2_collision.stl"/>
-        </geometry>
-      </collision>
-      <inertial>
-        <origin xyz="0 0 1" rpy="0 0 0"/>
-        <mass value="1"/>
-        <inertia
-      ixx="1" ixy="0.0" ixz="0.0"
-      iyy="1" iyz="0.0"
-      izz="1"/>
-      </inertial>
-    </link>
-  <link name="${prefix}link_2">
-      <visual>
-        <origin rpy="0 0 0" xyz="0 0 0"/>
-        <geometry>
-          <mesh filename="file://$(find manipulatorws)/meshes/pa10_stl/S3.stl"/>
-        </geometry>
-        <material name="">
-          <color rgba="0.34 0.35 0.36 1.0"/>
-        </material>
-      </visual>
-      <collision>
         <origin rpy="0 0 0" xyz="0 0 0"/>
         <geometry>
@@ -92,7 +92,6 @@
           <mesh filename="file://$(find manipulatorws)/meshes/pa10_stl/E1.stl"/>
         </geometry>
-    <material name="">
-          <color rgba="0.7 0.0 0.0 1.0"/>
-        </material>
+      <material name="">
+        <color rgba="0.0 1.0 1.0 0.4"/> <!-- RGB = Cyan, A = 30% visible -->      </material>
       </visual>
       <collision>
@@ -117,7 +116,7 @@
           <mesh filename="file://$(find manipulatorws)/meshes/pa10_stl/E2.stl"/>
         </geometry>
-    <material name="">
-          <color rgba="0.34 0.35 0.36 1.0"/>
-        </material>
+      <material name="">
+        <color rgba="0.0 1.0 1.0 0.4"/> <!-- RGB = Cyan, A = 30% visible -->
+      </material>
       </visual>
       <collision>
@@ -142,7 +141,7 @@
           <mesh filename="file://$(find manipulatorws)/meshes/pa10_stl/W1.stl"/>
         </geometry>
-    <material name="">
-          <color rgba="0.7 0.0 0.0 1.0"/>
-        </material>
+      <material name="">
+        <color rgba="0.0 1.0 1.0 0.4"/> <!-- RGB = Cyan, A = 30% visible -->
+      </material>
       </visual>
       <collision>
@@ -167,7 +166,7 @@
           <mesh filename="file://$(find manipulatorws)/meshes/pa10_stl/W2.stl"/>
         </geometry>
-    <material name="">
-          <color rgba="0.34 0.35 0.36 1.0"/>
-        </material>
+      <material name="hologram_cyan">
+        <color rgba="0.1 1.0 1.0 0.4"/> <!-- RGB = Cyan, A = 30% visible -->
+      </material>
       </visual>
       <collision>
@@ -200,5 +199,5 @@
         </geometry>
         <material name="">
-          <color rgba="0.8 0.0 0.0 1.0"/> <!-- red for visibility -->
+          <color rgba="0.0 1.0 1.0 0.5"/> <!-- RGB = Cyan, A = 30% visible -->
         </material>
       </visual>
@@ -225,5 +224,5 @@
                   </geometry>
                   <material name="">
-                    <color rgba="0.9 0.75 0.3 1.0"/>
+                    <color rgba="0.0 1.0 1.0 0.4"/> <!-- RGB = Cyan, A = 30% visible -->
                   </material>
               </visual>
@@ -250,5 +249,5 @@
                   </geometry>
                   <material name="">
-                    <color rgba="0.9 0.75 0.3 1.0"/>
+                    <color rgba="0.0 1.0 1.0 0.4"/> <!-- RGB = Cyan, A = 30% visible -->
                   </material>
               </visual>
